File: Eagle/Master/XBee_RPi_breakout.brd (EAGLE design)
At the start: 30 x 58 mm, 8 parts

Commit message: Backup changes
Other:
- board size 30 x 58 mm -> 28 x 56 mm
- board text removed: "/Users/ninjanymo/Desktop/logo.bmp"
Changed lines of the file:
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@@
 <layer number="19" name="Unrouted" color="6" fill="1" visible="no" active="yes"/>
 <layer number="20" name="Dimension" color="24" fill="1" visible="yes" active="yes"/>
-<layer number="21" name="tPlace" color="7" fill="1" visible="no" active="yes"/>
+<layer number="21" name="tPlace" color="7" fill="1" visible="yes" active="yes"/>
 <layer number="22" name="bPlace" color="7" fill="1" visible="no" active="yes"/>
 <layer number="23" name="tOrigins" color="15" fill="1" visible="no" active="yes"/>
@@
 <layer number="49" name="Reference" color="7" fill="1" visible="no" active="yes"/>
 <layer number="50" name="dxf" color="7" fill="1" visible="no" active="no"/>
-<layer number="51" name="tDocu" color="7" fill="1" visible="no" active="yes"/>
+<layer number="51" name="tDocu" color="7" fill="1" visible="yes" active="yes"/>
 <layer number="52" name="bDocu" color="7" fill="1" visible="no" active="yes"/>
 <layer number="53" name="tGND_GNDA" color="7" fill="9" visible="no" active="no"/>
@@
 <layer number="111" name="LPC17xx" color="7" fill="1" visible="no" active="yes"/>
 <layer number="112" name="tSilk" color="7" fill="1" visible="no" active="yes"/>
-<layer number="113" name="LOGO_TOP" color="1" fill="1" visible="yes" active="yes"/>
-<layer number="114" name="DRILLMARKS" color="12" fill="1" visible="yes" active="yes"/>
+<layer number="113" name="LOGO_TOP" color="4" fill="1" visible="yes" active="yes"/>
+<layer number="114" name="DRILLMARKS" color="12" fill="1" visible="no" active="yes"/>
 <layer number="116" name="Patch_BOT" color="9" fill="4" visible="no" active="yes"/>
 <layer number="121" name="_tsilk" color="7" fill="1" visible="no" active="yes"/>
@@
 <rectangle x1="7.9407" y1="6.29625" x2="8.8492" y2="6.30775" layer="113"/>
 <rectangle x1="7.9523" y1="6.30775" x2="8.8378" y2="6.31925" layer="113"/>
-<text x="5.474" y="1.0005" size="0.023" layer="113" font="vector">/Users/ninjanymo/Desktop/logo.bmp</text>
-<wire x1="-0.5" y1="-1" x2="0" y2="-1" width="0.6096" layer="20"/>
-<wire x1="0" y1="-1" x2="29" y2="-1" width="0.6096" layer="20"/>
-<wire x1="29" y1="57" x2="-1" y2="57" width="0.6096" layer="20"/>
-<wire x1="-1" y1="57" x2="-1" y2="-1" width="0.6096" layer="20"/>
-<wire x1="-1" y1="-1" x2="-0.5" y2="-1" width="0.6096" layer="20"/>
 </plain>
 <attributes>
